File: _autosave-555_Timer_Clock.kicad_pcb (KiCad board)
At the start: 2 copper layers, 39 x 25 mm, 13 parts, among them J2 CLK_Out, U1 ICM7555xB

Commit message: 555_timer_clock_finished design
Parts:
- added J1: +5V, my_footprints:Terminal_Block_5mm, F.Cu at (103.0, 72.5)
- added SW1: Trigger, my_footprints:slide_switch_2.54mm, F.Cu at (124.0, 81.5)
- added SW2: RST, my_footprints:tact_switch_5mm, F.Cu at (114.0, 81.5)
- moved R4 15.5 mm to (120.0, 65.5)
- moved R2 15.5 mm to (116.0, 65.5)
- moved R1 15.0 mm to (112.5, 65.5)
- moved D1 10.1 mm to (114.0, 72.5)
- moved R3 9.35 mm to (120.0, 74.5)
- moved C2 8.56 mm to (126.0, 66.0)
- moved U1 8.06 mm to (126.0, 73.5)
- moved J2 7.96 mm to (132.0, 71.8)
- moved C1 7.21 mm to (132.0, 75.2)
Routing:
- net GND: track 0.00 -> 72.8 mm, vias 0 -> 2
- net /+5V: track 0.00 -> 37.6 mm
- net /Trigger: track 0.00 -> 35.2 mm
- net /CLK_Out: track 0.00 -> 25.5 mm, vias 0 -> 1
- net /RST: track 0.00 -> 16.9 mm
- net Net-(U1-DISCH): track 0.00 -> 14.7 mm
- net Net-(D1-K): track 0.00 -> 9.34 mm
- net Net-(U1-CONT): track 0.00 -> 5.92 mm
